File: KiCAD/Tr_Vbe_AD2/Tr_Vbe_AD2.kicad_pcb (KiCad board)
At the start: 2 copper layers, 71.1 x 45.7 mm, 13 parts, among them J1 AD2, Q1 2SC1815, Q2 2SK170

Commit message: Update: Board design
Parts:
- moved RV1 2.54 mm to (152.4, 104.1)
Routing:
- net GND: track 67.8 -> 72.8 mm
- net Net-(Q2-Pad3): track 7.62 -> 8.67 mm
